File: kicad_source/rotaryencoder.kicad_sch (KiCad schematic)
At the start: 6 parts, among them U1 AS5048A, U2 AS5048A

Commit message: updated some symbol library links
Parts:
- C1, C2: renamed from C?; value (none) -> 100nF; footprint (none) -> capacitors:C_0603; symbol l3xz-leg-ctrl-hardware-rescue:C_0603-devices -> Device:C_Small
- R6, R7: renamed from R?; value (none) -> 10k; footprint (none) -> resistors:R_0603; symbol l3xz-leg-ctrl-hardware-rescue:R_0603-devices -> Device:R_Small
Connections:
- net +3V3 renamed +3.3V
Changed lines of the file:
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@@
   (title_block
     (title "l3xz-hw_leg-controller")
-    (date "2022-06-05")
+    (date "2023-01-26")
     (rev "dev_0.2")
     (company "107-systems")
@@
     )
   )
-  (symbol (lib_id "l3xz-leg-ctrl-hardware-rescue:R_0603-devices") (at 88.9 45.72 0) (unit 1)
-    (in_bom yes) (on_board yes)
-    (property "Reference" "R?" (id 0) (at 90.3986 44.5516 0)
-      (effects (font (size 1.27 1.27)) (justify left))
-    )
-    (property "Value" "" (id 1) (at 90.3986 46.863 0)
-      (effects (font (size 1.27 1.27)) (justify left))
-    )
-    (property "Footprint" "" (id 2) (at 88.9 49.53 0)
+  (symbol (lib_id "Device:R_Small") (at 88.9 45.72 0) (unit 1)
+    (in_bom yes) (on_board yes)
+    (property "Reference" "R6" (id 0) (at 90.3986 44.5516 0)
+      (effects (font (size 1.27 1.27)) (justify left))
+    )
+    (property "Value" "10k" (id 1) (at 90.3986 46.863 0)
+      (effects (font (size 1.27 1.27)) (justify left))
+    )
+    (property "Footprint" "resistors:R_0603" (id 2) (at 88.9 49.53 0)
       (effects (font (size 1.27 1.27)) hide)
     )
@@
     (pin "2")
   )
-  (symbol (lib_id "l3xz-leg-ctrl-hardware-rescue:+3.3V-power-supply") (at 88.9 41.91 0) (unit 1)
-    (in_bom yes) (on_board yes)
-    (property "Reference" "#PWR?" (id 0) (at 88.9 45.72 0)
-      (effects (font (size 1.27 1.27)) hide)
-    )
-    (property "Value" "" (id 1) (at 89.281 37.5158 0))
+  (symbol (lib_id "power:+3.3V") (at 88.9 41.91 0) (unit 1)
+    (in_bom yes) (on_board yes)
+    (property "Reference" "#PWR06" (id 0) (at 88.9 45.72 0)
+      (effects (font (size 1.27 1.27)) hide)
+    )
+    (property "Value" "+3.3V" (id 1) (at 89.281 37.5158 0))
     (property "Footprint" "" (id 2) (at 88.9 41.91 0))
     (property "Datasheet" "" (id 3) (at 88.9 41.91 0))
@@
     (pin "9")
   )
-  (symbol (lib_id "l3xz-leg-ctrl-hardware-rescue:C_0603-devices") (at 140.97 67.31 0) (unit 1)
-    (in_bom yes) (on_board yes)
-    (property "Reference" "C?" (id 0) (at 143.3068 66.1416 0)
-      (effects (font (size 1.27 1.27)) (justify left))
-    )
-    (property "Value" "" (id 1) (at 143.3068 68.453 0)
-      (effects (font (size 1.27 1.27)) (justify left))
-    )
-    (property "Footprint" "" (id 2) (at 140.97 71.12 0)
+  (symbol (lib_id "Device:C_Small") (at 140.97 67.31 0) (unit 1)
+    (in_bom yes) (on_board yes)
+    (property "Reference" "C1" (id 0) (at 143.3068 66.1416 0)
+      (effects (font (size 1.27 1.27)) (justify left))
+    )
+    (property "Value" "100nF" (id 1) (at 143.3068 68.453 0)
+      (effects (font (size 1.27 1.27)) (justify left))
+    )
+    (property "Footprint" "capacitors:C_0603" (id 2) (at 140.97 71.12 0)
       (effects (font (size 1.27 1.27)) hide)
     )
@@
     (pin "2")
   )
-  (symbol (lib_id "l3xz-leg-ctrl-hardware-rescue:+3.3V-power-supply") (at 140.97 62.23 0) (unit 1)
-    (in_bom yes) (on_board yes)
-    (property "Reference" "#PWR?" (id 0) (at 140.97 66.04 0)
-      (effects (font (size 1.27 1.27)) hide)
-    )
-    (property "Value" "" (id 1) (at 141.351 57.8358 0))
+  (symbol (lib_id "power:+3.3V") (at 140.97 62.23 0) (unit 1)
+    (in_bom yes) (on_board yes)
+    (property "Reference" "#PWR07" (id 0) (at 140.97 66.04 0)
+      (effects (font (size 1.27 1.27)) hide)
+    )
+    (property "Value" "+3.3V" (id 1) (at 141.351 57.8358 0))
     (property "Footprint" "" (id 2) (at 140.97 62.23 0))
     (property "Datasheet" "" (id 3) (at 140.97 62.23 0))
     (pin "1")
   )
-  (symbol (lib_id "l3xz-leg-ctrl-hardware-rescue:GND-power-supply") (at 140.97 71.12 0) (unit 1)
-    (in_bom yes) (on_board yes)
-    (property "Reference" "#PWR?" (id 0) (at 140.97 77.47 0)
-      (effects (font (size 1.27 1.27)) hide)
-    )
-    (property "Value" "" (id 1) (at 141.097 75.5142 0))
+  (symbol (lib_id "power:GND") (at 140.97 71.12 0) (unit 1)
+    (in_bom yes) (on_board yes)
+    (property "Reference" "#PWR09" (id 0) (at 140.97 77.47 0)
+      (effects (font (size 1.27 1.27)) hide)
+    )
+    (property "Value" "GND" (id 1) (at 141.097 75.5142 0))
     (property "Footprint" "" (id 2) (at 140.97 71.12 0))
     (property "Datasheet" "" (id 3) (at 140.97 71.12 0))
     (pin "1")
   )
-  (symbol (lib_id "l3xz-leg-ctrl-hardware-rescue:GND-power-supply") (at 97.79 71.12 0) (unit 1)
-    (in_bom yes) (on_board yes)
-    (property "Reference" "#PWR?" (id 0) (at 97.79 77.47 0)
-      (effects (font (size 1.27 1.27)) hide)
-    )
-    (property "Value" "" (id 1) (at 97.917 75.5142 0))
+  (symbol (lib_id "power:GND") (at 97.79 71.12 0) (unit 1)
+    (in_bom yes) (on_board yes)
+    (property "Reference" "#PWR08" (id 0) (at 97.79 77.47 0)
+      (effects (font (size 1.27 1.27)) hide)
+    )
+    (property "Value" "GND" (id 1) (at 97.917 75.5142 0))
     (property "Footprint" "" (id 2) (at 97.79 71.12 0))
     (property "Datasheet" "" (id 3) (at 97.79 71.12 0))
     (pin "1")
   )
-  (symbol (lib_id "l3xz-leg-ctrl-hardware-rescue:R_0603-devices") (at 88.9 107.95 0) (unit 1)
-    (in_bom yes) (on_board yes)
-    (property "Reference" "R?" (id 0) (at 90.3986 106.7816 0)
-      (effects (font (size 1.27 1.27)) (justify left))
-    )
-    (property "Value" "" (id 1) (at 90.3986 109.093 0)
-      (effects (font (size 1.27 1.27)) (justify left))
-    )
-    (property "Footprint" "" (id 2) (at 88.9 111.76 0)
+  (symbol (lib_id "Device:R_Small") (at 88.9 107.95 0) (unit 1)
+    (in_bom yes) (on_board yes)
+    (property "Reference" "R7" (id 0) (at 90.3986 106.7816 0)
+      (effects (font (size 1.27 1.27)) (justify left))
+    )
+    (property "Value" "10k" (id 1) (at 90.3986 109.093 0)
+      (effects (font (size 1.27 1.27)) (justify left))
+    )
+    (property "Footprint" "resistors:R_0603" (id 2) (at 88.9 111.76 0)
       (effects (font (size 1.27 1.27)) hide)
     )
@@
     (pin "2")
   )
-  (symbol (lib_id "l3xz-leg-ctrl-hardware-rescue:+3.3V-power-supply") (at 88.9 104.14 0) (unit 1)
-    (in_bom yes) (on_board yes)
-    (property "Reference" "#PWR?" (id 0) (at 88.9 107.95 0)
-      (effects (font (size 1.27 1.27)) hide)
-    )
-    (property "Value" "" (id 1) (at 89.281 99.7458 0))
+  (symbol (lib_id "power:+3.3V") (at 88.9 104.14 0) (unit 1)
+    (in_bom yes) (on_board yes)
+    (property "Reference" "#PWR010" (id 0) (at 88.9 107.95 0)
+      (effects (font (size 1.27 1.27)) hide)
+    )
+    (property "Value" "+3.3V" (id 1) (at 89.281 99.7458 0))
     (property "Footprint" "" (id 2) (at 88.9 104.14 0))
     (property "Datasheet" "" (id 3) (at 88.9 104.14 0))
@@
     (pin "9")
   )
-  (symbol (lib_id "l3xz-leg-ctrl-hardware-rescue:C_0603-devices") (at 140.97 129.54 0) (unit 1)
-    (in_bom yes) (on_board yes)
-    (property "Reference" "C?" (id 0) (at 143.3068 128.3716 0)
-      (effects (font (size 1.27 1.27)) (justify left))
-    )
-    (property "Value" "" (id 1) (at 143.3068 130.683 0)
-      (effects (font (size 1.27 1.27)) (justify left))
-    )
-    (property "Footprint" "" (id 2) (at 140.97 133.35 0)
+  (symbol (lib_id "Device:C_Small") (at 140.97 129.54 0) (unit 1)
+    (in_bom yes) (on_board yes)
+    (property "Reference" "C2" (id 0) (at 143.3068 128.3716 0)
+      (effects (font (size 1.27 1.27)) (justify left))
+    )
+    (property "Value" "100nF" (id 1) (at 143.3068 130.683 0)
+      (effects (font (size 1.27 1.27)) (justify left))
+    )
+    (property "Footprint" "capacitors:C_0603" (id 2) (at 140.97 133.35 0)
       (effects (font (size 1.27 1.27)) hide)
     )
@@
     (pin "2")
   )
-  (symbol (lib_id "l3xz-leg-ctrl-hardware-rescue:+3.3V-power-supply") (at 140.97 124.46 0) (unit 1)
-    (in_bom yes) (on_board yes)
-    (property "Reference" "#PWR?" (id 0) (at 140.97 128.27 0)
-      (effects (font (size 1.27 1.27)) hide)
-    )
-    (property "Value" "" (id 1) (at 141.351 120.0658 0))
+  (symbol (lib_id "power:+3.3V") (at 140.97 124.46 0) (unit 1)
+    (in_bom yes) (on_board yes)
+    (property "Reference" "#PWR011" (id 0) (at 140.97 128.27 0)
+      (effects (font (size 1.27 1.27)) hide)
+    )
+    (property "Value" "+3.3V" (id 1) (at 141.351 120.0658 0))
     (property "Footprint" "" (id 2) (at 140.97 124.46 0))
     (property "Datasheet" "" (id 3) (at 140.97 124.46 0))
     (pin "1")
   )
-  (symbol (lib_id "l3xz-leg-ctrl-hardware-rescue:GND-power-supply") (at 140.97 133.35 0) (unit 1)
-    (in_bom yes) (on_board yes)
-    (property "Reference" "#PWR?" (id 0) (at 140.97 139.7 0)
-      (effects (font (size 1.27 1.27)) hide)
-    )
-    (property "Value" "" (id 1) (at 141.097 137.7442 0))
+  (symbol (lib_id "power:GND") (at 140.97 133.35 0) (unit 1)
+    (in_bom yes) (on_board yes)
+    (property "Reference" "#PWR013" (id 0) (at 140.97 139.7 0)
+      (effects (font (size 1.27 1.27)) hide)
+    )
+    (property "Value" "GND" (id 1) (at 141.097 137.7442 0))
     (property "Footprint" "" (id 2) (at 140.97 133.35 0))
     (property "Datasheet" "" (id 3) (at 140.97 133.35 0))
     (pin "1")
   )
-  (symbol (lib_id "l3xz-leg-ctrl-hardware-rescue:GND-power-supply") (at 97.79 133.35 0) (unit 1)
-    (in_bom yes) (on_board yes)
-    (property "Reference" "#PWR?" (id 0) (at 97.79 139.7 0)
-      (effects (font (size 1.27 1.27)) hide)
-    )
-    (property "Value" "" (id 1) (at 97.917 137.7442 0))
+  (symbol (lib_id "power:GND") (at 97.79 133.35 0) (unit 1)
+    (in_bom yes) (on_board yes)
+    (property "Reference" "#PWR012" (id 0) (at 97.79 139.7 0)
+      (effects (font (size 1.27 1.27)) hide)
+    )
+    (property "Value" "GND" (id 1) (at 97.917 137.7442 0))
     (property "Footprint" "" (id 2) (at 97.79 133.35 0))
     (property "Datasheet" "" (id 3) (at 97.79 133.35 0))

Commit message: updated footprint library
Parts:
- C1, C2: footprint capacitors:C_0603 -> Capacitor_SMD:C_0603_1608Metric
- R6, R7: footprint resistors:R_0603 -> Resistor_SMD:R_0603_1608Metric
- U1, U2: footprint SSOP:TSSOP-14_4.4x5mm_Pitch0.65mm -> Package_SO:TSSOP-14_4.4x5mm_P0.65mm
Changed lines of the file:
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@@
   (title_block
     (title "l3xz-hw_leg-controller")
-    (date "2023-01-26")
+    (date "2023-01-29")
     (rev "dev_0.2")
     (company "107-systems")
@@
       (effects (font (size 1.27 1.27)) (justify left))
     )
-    (property "Footprint" "resistors:R_0603" (id 2) (at 88.9 49.53 0)
+    (property "Footprint" "Resistor_SMD:R_0603_1608Metric" (id 2) (at 88.9 49.53 0)
       (effects (font (size 1.27 1.27)) hide)
     )
@@
       (effects (font (size 1.524 1.524)))
     )
-    (property "Footprint" "SSOP:TSSOP-14_4.4x5mm_Pitch0.65mm" (id 2) (at 115.57 53.34 0)
+    (property "Footprint" "Package_SO:TSSOP-14_4.4x5mm_P0.65mm" (id 2) (at 115.57 53.34 0)
       (effects (font (size 1.524 1.524)) hide)
     )
@@
       (effects (font (size 1.27 1.27)) (justify left))
     )
-    (property "Footprint" "capacitors:C_0603" (id 2) (at 140.97 71.12 0)
+    (property "Footprint" "Capacitor_SMD:C_0603_1608Metric" (id 2) (at 140.97 71.12 0)
       (effects (font (size 1.27 1.27)) hide)
     )
@@
       (effects (font (size 1.27 1.27)) (justify left))
     )
-    (property "Footprint" "resistors:R_0603" (id 2) (at 88.9 111.76 0)
+    (property "Footprint" "Resistor_SMD:R_0603_1608Metric" (id 2) (at 88.9 111.76 0)
       (effects (font (size 1.27 1.27)) hide)
     )
@@
       (effects (font (size 1.524 1.524)))
     )
-    (property "Footprint" "SSOP:TSSOP-14_4.4x5mm_Pitch0.65mm" (id 2) (at 115.57 115.57 0)
+    (property "Footprint" "Package_SO:TSSOP-14_4.4x5mm_P0.65mm" (id 2) (at 115.57 115.57 0)
       (effects (font (size 1.524 1.524)) hide)
     )
@@
       (effects (font (size 1.27 1.27)) (justify left))
     )
-    (property "Footprint" "capacitors:C_0603" (id 2) (at 140.97 133.35 0)
-      (effects (font (size 1.27 1.27)) hide)
-    )
+    (property "Footprint" "Capacitor_SMD:C_0603_1608Metric" (id 2) (at 140.97 133.35 0)
+      (effects (font (size 1.27 1.27)) hide)
+    )
